Commit message: support rox-argo-trio

File: neo_ur_moveit_config/srdf/rox.srdf.xacro (robot description, xacro)
@@ -6,5 +6,7 @@
 <robot xmlns:xacro="http://www.ros.org/wiki/xacro" name="rox">
      <xacro:arg name="prefix" default=""/>
+     <xacro:arg name="rox_type" default="argo"/>
      <xacro:property name="prefix_value" value="$(arg prefix)"/>
+     <xacro:property name="rox_typ" value="$(arg rox_type)"/>
     <!--GROUPS: Representation of a set of joints and links. This can be useful for specifying DOF to plan for, defining arms, end effectors, etc-->
     <!--LINKS: When a link is specified, the parent joint of that link (if it exists) is automatically included-->
@@ -25,111 +27,196 @@
     <disable_collisions link1="base_footprint" link2="lidar_1_link" reason="Adjacent"/>
     <disable_collisions link1="base_footprint" link2="lidar_2_link" reason="Adjacent"/>
-    <disable_collisions link1="base_footprint" link2="caster_back_left_link" reason="Adjacent"/>
-    <disable_collisions link1="base_footprint" link2="caster_back_right_link" reason="Adjacent"/>
-    <disable_collisions link1="base_footprint" link2="caster_front_left_link" reason="Adjacent"/>
-    <disable_collisions link1="base_footprint" link2="caster_front_right_link" reason="Adjacent"/>
-    <disable_collisions link1="base_footprint" link2="wheel_back_left_link" reason="Never"/>
-    <disable_collisions link1="base_footprint" link2="wheel_back_right_link" reason="Never"/>
-    <disable_collisions link1="base_footprint" link2="wheel_front_left_link" reason="Never"/>
-    <disable_collisions link1="base_footprint" link2="wheel_front_right_link" reason="Never"/>
-    <disable_collisions link1="base_footprint" link2="${prefix_value}base_link_inertia" reason="Never"/>
-    <disable_collisions link1="base_footprint" link2="${prefix_value}shoulder_link" reason="Never"/>
-    <disable_collisions link1="cabinet_link" link2="lidar_1_link" reason="Adjacent"/>
-    <disable_collisions link1="cabinet_link" link2="lidar_2_link" reason="Adjacent"/>
-    <disable_collisions link1="cabinet_link" link2="caster_back_left_link" reason="Never"/>
-    <disable_collisions link1="cabinet_link" link2="caster_back_right_link" reason="Never"/>
-    <disable_collisions link1="cabinet_link" link2="caster_front_left_link" reason="Never"/>
-    <disable_collisions link1="cabinet_link" link2="caster_front_right_link" reason="Never"/>
-    <disable_collisions link1="cabinet_link" link2="wheel_back_left_link" reason="Never"/>
-    <disable_collisions link1="cabinet_link" link2="wheel_back_right_link" reason="Never"/>
-    <disable_collisions link1="cabinet_link" link2="wheel_front_left_link" reason="Never"/>
-    <disable_collisions link1="cabinet_link" link2="wheel_front_right_link" reason="Never"/>
-    <disable_collisions link1="cabinet_link" link2="${prefix_value}base_link_inertia" reason="Adjacent"/>
-    <disable_collisions link1="cabinet_link" link2="${prefix_value}shoulder_link" reason="Never"/>
-    <disable_collisions link1="lidar_1_link" link2="lidar_2_link" reason="Adjacent"/>
-    <disable_collisions link1="lidar_1_link" link2="caster_back_left_link" reason="Never"/>
-    <disable_collisions link1="lidar_1_link" link2="caster_back_right_link" reason="Never"/>
-    <disable_collisions link1="lidar_1_link" link2="caster_front_left_link" reason="Never"/>
-    <disable_collisions link1="lidar_1_link" link2="caster_front_right_link" reason="Never"/>
-    <disable_collisions link1="lidar_1_link" link2="wheel_back_left_link" reason="Never"/>
-    <disable_collisions link1="lidar_1_link" link2="wheel_back_right_link" reason="Never"/>
-    <disable_collisions link1="lidar_1_link" link2="wheel_front_left_link" reason="Never"/>
-    <disable_collisions link1="lidar_1_link" link2="wheel_front_right_link" reason="Never"/>
-    <disable_collisions link1="lidar_1_link" link2="${prefix_value}base_link_inertia" reason="Never"/>
-    <disable_collisions link1="lidar_1_link" link2="${prefix_value}shoulder_link" reason="Never"/>
-    <disable_collisions link1="lidar_2_link" link2="caster_back_left_link" reason="Never"/>
-    <disable_collisions link1="lidar_2_link" link2="caster_back_right_link" reason="Never"/>
-    <disable_collisions link1="lidar_2_link" link2="caster_front_left_link" reason="Never"/>
-    <disable_collisions link1="lidar_2_link" link2="caster_front_right_link" reason="Never"/>
-    <disable_collisions link1="lidar_2_link" link2="wheel_back_left_link" reason="Never"/>
-    <disable_collisions link1="lidar_2_link" link2="wheel_back_right_link" reason="Never"/>
-    <disable_collisions link1="lidar_2_link" link2="wheel_front_left_link" reason="Never"/>
-    <disable_collisions link1="lidar_2_link" link2="wheel_front_right_link" reason="Never"/>
-    <disable_collisions link1="lidar_2_link" link2="${prefix_value}base_link_inertia" reason="Never"/>
-    <disable_collisions link1="lidar_2_link" link2="${prefix_value}shoulder_link" reason="Never"/>
-    <disable_collisions link1="lidar_2_link" link2="${prefix_value}upper_arm_link" reason="Never"/>
-    <disable_collisions link1="caster_back_left_link" link2="caster_back_right_link" reason="Never"/>
-    <disable_collisions link1="caster_back_left_link" link2="caster_front_left_link" reason="Never"/>
-    <disable_collisions link1="caster_back_left_link" link2="caster_front_right_link" reason="Never"/>
-    <disable_collisions link1="caster_back_left_link" link2="wheel_back_left_link" reason="Adjacent"/>
-    <disable_collisions link1="caster_back_left_link" link2="wheel_back_right_link" reason="Never"/>
-    <disable_collisions link1="caster_back_left_link" link2="wheel_front_left_link" reason="Never"/>
-    <disable_collisions link1="caster_back_left_link" link2="wheel_front_right_link" reason="Never"/>
-    <disable_collisions link1="caster_back_left_link" link2="${prefix_value}base_link_inertia" reason="Never"/>
-    <disable_collisions link1="caster_back_left_link" link2="${prefix_value}shoulder_link" reason="Never"/>
-    <disable_collisions link1="caster_back_left_link" link2="${prefix_value}upper_arm_link" reason="Never"/>
-    <disable_collisions link1="caster_back_right_link" link2="caster_front_left_link" reason="Never"/>
-    <disable_collisions link1="caster_back_right_link" link2="caster_front_right_link" reason="Never"/>
-    <disable_collisions link1="caster_back_right_link" link2="wheel_back_left_link" reason="Never"/>
-    <disable_collisions link1="caster_back_right_link" link2="wheel_back_right_link" reason="Adjacent"/>
-    <disable_collisions link1="caster_back_right_link" link2="wheel_front_left_link" reason="Never"/>
-    <disable_collisions link1="caster_back_right_link" link2="wheel_front_right_link" reason="Never"/>
-    <disable_collisions link1="caster_back_right_link" link2="${prefix_value}base_link_inertia" reason="Never"/>
-    <disable_collisions link1="caster_back_right_link" link2="${prefix_value}shoulder_link" reason="Never"/>
-    <disable_collisions link1="caster_back_right_link" link2="${prefix_value}upper_arm_link" reason="Never"/>
-    <disable_collisions link1="caster_front_left_link" link2="caster_front_right_link" reason="Never"/>
-    <disable_collisions link1="caster_front_left_link" link2="wheel_back_left_link" reason="Never"/>
-    <disable_collisions link1="caster_front_left_link" link2="wheel_back_right_link" reason="Never"/>
-    <disable_collisions link1="caster_front_left_link" link2="wheel_front_left_link" reason="Adjacent"/>
-    <disable_collisions link1="caster_front_left_link" link2="wheel_front_right_link" reason="Never"/>
-    <disable_collisions link1="caster_front_left_link" link2="${prefix_value}base_link_inertia" reason="Never"/>
-    <disable_collisions link1="caster_front_left_link" link2="${prefix_value}shoulder_link" reason="Never"/>
-    <disable_collisions link1="caster_front_right_link" link2="wheel_back_left_link" reason="Never"/>
-    <disable_collisions link1="caster_front_right_link" link2="wheel_back_right_link" reason="Never"/>
-    <disable_collisions link1="caster_front_right_link" link2="wheel_front_left_link" reason="Never"/>
-    <disable_collisions link1="caster_front_right_link" link2="wheel_front_right_link" reason="Adjacent"/>
-    <disable_collisions link1="caster_front_right_link" link2="${prefix_value}base_link_inertia" reason="Never"/>
-    <disable_collisions link1="caster_front_right_link" link2="${prefix_value}shoulder_link" reason="Never"/>
-    <disable_collisions link1="wheel_back_left_link" link2="wheel_back_right_link" reason="Never"/>
-    <disable_collisions link1="wheel_back_left_link" link2="wheel_front_left_link" reason="Never"/>
-    <disable_collisions link1="wheel_back_left_link" link2="wheel_front_right_link" reason="Never"/>
-    <disable_collisions link1="wheel_back_left_link" link2="${prefix_value}base_link_inertia" reason="Never"/>
-    <disable_collisions link1="wheel_back_left_link" link2="${prefix_value}shoulder_link" reason="Never"/>
-    <disable_collisions link1="wheel_back_left_link" link2="${prefix_value}upper_arm_link" reason="Never"/>
-    <disable_collisions link1="wheel_back_right_link" link2="wheel_front_left_link" reason="Never"/>
-    <disable_collisions link1="wheel_back_right_link" link2="wheel_front_right_link" reason="Never"/>
-    <disable_collisions link1="wheel_back_right_link" link2="${prefix_value}base_link_inertia" reason="Never"/>
-    <disable_collisions link1="wheel_back_right_link" link2="${prefix_value}shoulder_link" reason="Never"/>
-    <disable_collisions link1="wheel_back_right_link" link2="${prefix_value}upper_arm_link" reason="Never"/>
-    <disable_collisions link1="wheel_front_left_link" link2="wheel_front_right_link" reason="Never"/>
-    <disable_collisions link1="wheel_front_left_link" link2="${prefix_value}base_link_inertia" reason="Never"/>
-    <disable_collisions link1="wheel_front_left_link" link2="${prefix_value}shoulder_link" reason="Never"/>
-    <disable_collisions link1="wheel_front_left_link" link2="${prefix_value}upper_arm_link" reason="Never"/>
-    <disable_collisions link1="wheel_front_right_link" link2="${prefix_value}base_link_inertia" reason="Never"/>
-    <disable_collisions link1="wheel_front_right_link" link2="${prefix_value}shoulder_link" reason="Never"/>
-    <disable_collisions link1="wheel_front_right_link" link2="${prefix_value}upper_arm_link" reason="Never"/>
-    <disable_collisions link1="${prefix_value}base_link_inertia" link2="${prefix_value}shoulder_link" reason="Adjacent"/>
-    <disable_collisions link1="${prefix_value}base_link_inertia" link2="${prefix_value}upper_arm_link" reason="Never"/>
-    <disable_collisions link1="${prefix_value}base_link_inertia" link2="${prefix_value}wrist_1_link" reason="Never"/>
-    <disable_collisions link1="${prefix_value}forearm_link" link2="${prefix_value}upper_arm_link" reason="Adjacent"/>
-    <disable_collisions link1="${prefix_value}forearm_link" link2="${prefix_value}wrist_1_link" reason="Adjacent"/>
-    <disable_collisions link1="${prefix_value}shoulder_link" link2="${prefix_value}upper_arm_link" reason="Adjacent"/>
-    <disable_collisions link1="${prefix_value}shoulder_link" link2="${prefix_value}wrist_1_link" reason="Never"/>
-    <disable_collisions link1="${prefix_value}shoulder_link" link2="${prefix_value}wrist_2_link" reason="Never"/>
-    <disable_collisions link1="${prefix_value}wrist_1_link" link2="${prefix_value}wrist_2_link" reason="Adjacent"/>
-    <disable_collisions link1="${prefix_value}wrist_1_link" link2="${prefix_value}wrist_3_link" reason="Never"/>
-    <disable_collisions link1="${prefix_value}wrist_2_link" link2="${prefix_value}wrist_3_link" reason="Adjacent"/>
-    <disable_collisions link1="${prefix_value}tool0" link2="${prefix_value}wrist_1_link" reason="Never" />
-    <disable_collisions link1="${prefix_value}tool0" link2="${prefix_value}wrist_2_link" reason="Never" />
-    <disable_collisions link1="${prefix_value}tool0" link2="${prefix_value}wrist_3_link" reason="Adjacent" />
+    <xacro:if value="${rox_typ == 'argo'}">
+        <disable_collisions link1="base_footprint" link2="caster_back_left_link" reason="Adjacent"/>
+        <disable_collisions link1="base_footprint" link2="caster_back_right_link" reason="Adjacent"/>
+        <disable_collisions link1="base_footprint" link2="caster_front_left_link" reason="Adjacent"/>
+        <disable_collisions link1="base_footprint" link2="caster_front_right_link" reason="Adjacent"/>
+        <disable_collisions link1="base_footprint" link2="wheel_back_left_link" reason="Never"/>
+        <disable_collisions link1="base_footprint" link2="wheel_back_right_link" reason="Never"/>
+        <disable_collisions link1="base_footprint" link2="wheel_front_left_link" reason="Never"/>
+        <disable_collisions link1="base_footprint" link2="wheel_front_right_link" reason="Never"/>
+        <disable_collisions link1="base_footprint" link2="${prefix_value}base_link_inertia" reason="Never"/>
+        <disable_collisions link1="base_footprint" link2="${prefix_value}shoulder_link" reason="Never"/>
+        <disable_collisions link1="cabinet_link" link2="lidar_1_link" reason="Adjacent"/>
+        <disable_collisions link1="cabinet_link" link2="lidar_2_link" reason="Adjacent"/>
+        <disable_collisions link1="cabinet_link" link2="caster_back_left_link" reason="Never"/>
+        <disable_collisions link1="cabinet_link" link2="caster_back_right_link" reason="Never"/>
+        <disable_collisions link1="cabinet_link" link2="caster_front_left_link" reason="Never"/>
+        <disable_collisions link1="cabinet_link" link2="caster_front_right_link" reason="Never"/>
+        <disable_collisions link1="cabinet_link" link2="wheel_back_left_link" reason="Never"/>
+        <disable_collisions link1="cabinet_link" link2="wheel_back_right_link" reason="Never"/>
+        <disable_collisions link1="cabinet_link" link2="wheel_front_left_link" reason="Never"/>
+        <disable_collisions link1="cabinet_link" link2="wheel_front_right_link" reason="Never"/>
+        <disable_collisions link1="cabinet_link" link2="${prefix_value}base_link_inertia" reason="Adjacent"/>
+        <disable_collisions link1="cabinet_link" link2="${prefix_value}shoulder_link" reason="Never"/>
+        <disable_collisions link1="lidar_1_link" link2="lidar_2_link" reason="Adjacent"/>
+        <disable_collisions link1="lidar_1_link" link2="caster_back_left_link" reason="Never"/>
+        <disable_collisions link1="lidar_1_link" link2="caster_back_right_link" reason="Never"/>
+        <disable_collisions link1="lidar_1_link" link2="caster_front_left_link" reason="Never"/>
+        <disable_collisions link1="lidar_1_link" link2="caster_front_right_link" reason="Never"/>
+        <disable_collisions link1="lidar_1_link" link2="wheel_back_left_link" reason="Never"/>
+        <disable_collisions link1="lidar_1_link" link2="wheel_back_right_link" reason="Never"/>
+        <disable_collisions link1="lidar_1_link" link2="wheel_front_left_link" reason="Never"/>
+        <disable_collisions link1="lidar_1_link" link2="wheel_front_right_link" reason="Never"/>
+        <disable_collisions link1="lidar_1_link" link2="${prefix_value}base_link_inertia" reason="Never"/>
+        <disable_collisions link1="lidar_1_link" link2="${prefix_value}shoulder_link" reason="Never"/>
+        <disable_collisions link1="lidar_2_link" link2="caster_back_left_link" reason="Never"/>
+        <disable_collisions link1="lidar_2_link" link2="caster_back_right_link" reason="Never"/>
+        <disable_collisions link1="lidar_2_link" link2="caster_front_left_link" reason="Never"/>
+        <disable_collisions link1="lidar_2_link" link2="caster_front_right_link" reason="Never"/>
+        <disable_collisions link1="lidar_2_link" link2="wheel_back_left_link" reason="Never"/>
+        <disable_collisions link1="lidar_2_link" link2="wheel_back_right_link" reason="Never"/>
+        <disable_collisions link1="lidar_2_link" link2="wheel_front_left_link" reason="Never"/>
+        <disable_collisions link1="lidar_2_link" link2="wheel_front_right_link" reason="Never"/>
+        <disable_collisions link1="lidar_2_link" link2="${prefix_value}base_link_inertia" reason="Never"/>
+        <disable_collisions link1="lidar_2_link" link2="${prefix_value}shoulder_link" reason="Never"/>
+        <disable_collisions link1="lidar_2_link" link2="${prefix_value}upper_arm_link" reason="Never"/>
+        <disable_collisions link1="caster_back_left_link" link2="caster_back_right_link" reason="Never"/>
+        <disable_collisions link1="caster_back_left_link" link2="caster_front_left_link" reason="Never"/>
+        <disable_collisions link1="caster_back_left_link" link2="caster_front_right_link" reason="Never"/>
+        <disable_collisions link1="caster_back_left_link" link2="wheel_back_left_link" reason="Adjacent"/>
+        <disable_collisions link1="caster_back_left_link" link2="wheel_back_right_link" reason="Never"/>
+        <disable_collisions link1="caster_back_left_link" link2="wheel_front_left_link" reason="Never"/>
+        <disable_collisions link1="caster_back_left_link" link2="wheel_front_right_link" reason="Never"/>
+        <disable_collisions link1="caster_back_left_link" link2="${prefix_value}base_link_inertia" reason="Never"/>
+        <disable_collisions link1="caster_back_left_link" link2="${prefix_value}shoulder_link" reason="Never"/>
+        <disable_collisions link1="caster_back_left_link" link2="${prefix_value}upper_arm_link" reason="Never"/>
+        <disable_collisions link1="caster_back_right_link" link2="caster_front_left_link" reason="Never"/>
+        <disable_collisions link1="caster_back_right_link" link2="caster_front_right_link" reason="Never"/>
+        <disable_collisions link1="caster_back_right_link" link2="wheel_back_left_link" reason="Never"/>
+        <disable_collisions link1="caster_back_right_link" link2="wheel_back_right_link" reason="Adjacent"/>
+        <disable_collisions link1="caster_back_right_link" link2="wheel_front_left_link" reason="Never"/>
+        <disable_collisions link1="caster_back_right_link" link2="wheel_front_right_link" reason="Never"/>
+        <disable_collisions link1="caster_back_right_link" link2="${prefix_value}base_link_inertia" reason="Never"/>
+        <disable_collisions link1="caster_back_right_link" link2="${prefix_value}shoulder_link" reason="Never"/>
+        <disable_collisions link1="caster_back_right_link" link2="${prefix_value}upper_arm_link" reason="Never"/>
+        <disable_collisions link1="caster_front_left_link" link2="caster_front_right_link" reason="Never"/>
+        <disable_collisions link1="caster_front_left_link" link2="wheel_back_left_link" reason="Never"/>
+        <disable_collisions link1="caster_front_left_link" link2="wheel_back_right_link" reason="Never"/>
+        <disable_collisions link1="caster_front_left_link" link2="wheel_front_left_link" reason="Adjacent"/>
+        <disable_collisions link1="caster_front_left_link" link2="wheel_front_right_link" reason="Never"/>
+        <disable_collisions link1="caster_front_left_link" link2="${prefix_value}base_link_inertia" reason="Never"/>
+        <disable_collisions link1="caster_front_left_link" link2="${prefix_value}shoulder_link" reason="Never"/>
+        <disable_collisions link1="caster_front_right_link" link2="wheel_back_left_link" reason="Never"/>
+        <disable_collisions link1="caster_front_right_link" link2="wheel_back_right_link" reason="Never"/>
+        <disable_collisions link1="caster_front_right_link" link2="wheel_front_left_link" reason="Never"/>
+        <disable_collisions link1="caster_front_right_link" link2="wheel_front_right_link" reason="Adjacent"/>
+        <disable_collisions link1="caster_front_right_link" link2="${prefix_value}base_link_inertia" reason="Never"/>
+        <disable_collisions link1="caster_front_right_link" link2="${prefix_value}shoulder_link" reason="Never"/>
+        <disable_collisions link1="wheel_back_left_link" link2="wheel_back_right_link" reason="Never"/>
+        <disable_collisions link1="wheel_back_left_link" link2="wheel_front_left_link" reason="Never"/>
+        <disable_collisions link1="wheel_back_left_link" link2="wheel_front_right_link" reason="Never"/>
+        <disable_collisions link1="wheel_back_left_link" link2="${prefix_value}base_link_inertia" reason="Never"/>
+        <disable_collisions link1="wheel_back_left_link" link2="${prefix_value}shoulder_link" reason="Never"/>
+        <disable_collisions link1="wheel_back_left_link" link2="${prefix_value}upper_arm_link" reason="Never"/>
+        <disable_collisions link1="wheel_back_right_link" link2="wheel_front_left_link" reason="Never"/>
+        <disable_collisions link1="wheel_back_right_link" link2="wheel_front_right_link" reason="Never"/>
+        <disable_collisions link1="wheel_back_right_link" link2="${prefix_value}base_link_inertia" reason="Never"/>
+        <disable_collisions link1="wheel_back_right_link" link2="${prefix_value}shoulder_link" reason="Never"/>
+        <disable_collisions link1="wheel_back_right_link" link2="${prefix_value}upper_arm_link" reason="Never"/>
+        <disable_collisions link1="wheel_front_left_link" link2="wheel_front_right_link" reason="Never"/>
+        <disable_collisions link1="wheel_front_left_link" link2="${prefix_value}base_link_inertia" reason="Never"/>
+        <disable_collisions link1="wheel_front_left_link" link2="${prefix_value}shoulder_link" reason="Never"/>
+        <disable_collisions link1="wheel_front_left_link" link2="${prefix_value}upper_arm_link" reason="Never"/>
+        <disable_collisions link1="wheel_front_right_link" link2="${prefix_value}base_link_inertia" reason="Never"/>
+        <disable_collisions link1="wheel_front_right_link" link2="${prefix_value}shoulder_link" reason="Never"/>
+        <disable_collisions link1="wheel_front_right_link" link2="${prefix_value}upper_arm_link" reason="Never"/>
+        <disable_collisions link1="${prefix_value}base_link_inertia" link2="${prefix_value}shoulder_link" reason="Adjacent"/>
+        <disable_collisions link1="${prefix_value}base_link_inertia" link2="${prefix_value}upper_arm_link" reason="Never"/>
+        <disable_collisions link1="${prefix_value}base_link_inertia" link2="${prefix_value}wrist_1_link" reason="Never"/>
+        <disable_collisions link1="${prefix_value}forearm_link" link2="${prefix_value}upper_arm_link" reason="Adjacent"/>
+        <disable_collisions link1="${prefix_value}forearm_link" link2="${prefix_value}wrist_1_link" reason="Adjacent"/>
+        <disable_collisions link1="${prefix_value}shoulder_link" link2="${prefix_value}upper_arm_link" reason="Adjacent"/>
+        <disable_collisions link1="${prefix_value}shoulder_link" link2="${prefix_value}wrist_1_link" reason="Never"/>
+        <disable_collisions link1="${prefix_value}shoulder_link" link2="${prefix_value}wrist_2_link" reason="Never"/>
+        <disable_collisions link1="${prefix_value}wrist_1_link" link2="${prefix_value}wrist_2_link" reason="Adjacent"/>
+        <disable_collisions link1="${prefix_value}wrist_1_link" link2="${prefix_value}wrist_3_link" reason="Never"/>
+        <disable_collisions link1="${prefix_value}wrist_2_link" link2="${prefix_value}wrist_3_link" reason="Adjacent"/>
+        <disable_collisions link1="${prefix_value}tool0" link2="${prefix_value}wrist_1_link" reason="Never" />
+        <disable_collisions link1="${prefix_value}tool0" link2="${prefix_value}wrist_2_link" reason="Never" />
+        <disable_collisions link1="${prefix_value}tool0" link2="${prefix_value}wrist_3_link" reason="Adjacent" />
+    </xacro:if>
+    <xacro:if value="${rox_typ == 'argo-trio'}">
+        <disable_collisions link1="base_footprint" link2="caster_back_link" reason="Adjacent"/>
+        <disable_collisions link1="base_footprint" link2="caster_front_left_link" reason="Adjacent"/>
+        <disable_collisions link1="base_footprint" link2="caster_front_right_link" reason="Adjacent"/>
+        <disable_collisions link1="base_footprint" link2="wheel_back_link" reason="Never"/>
+        <disable_collisions link1="base_footprint" link2="wheel_front_left_link" reason="Never"/>
+        <disable_collisions link1="base_footprint" link2="wheel_front_right_link" reason="Never"/>
+        <disable_collisions link1="base_footprint" link2="${prefix_value}base_link_inertia" reason="Never"/>
+        <disable_collisions link1="base_footprint" link2="${prefix_value}shoulder_link" reason="Never"/>
+        <disable_collisions link1="cabinet_link" link2="lidar_1_link" reason="Adjacent"/>
+        <disable_collisions link1="cabinet_link" link2="lidar_2_link" reason="Adjacent"/>
+        <disable_collisions link1="cabinet_link" link2="caster_back_link" reason="Never"/>
+        <disable_collisions link1="cabinet_link" link2="caster_front_left_link" reason="Never"/>
+        <disable_collisions link1="cabinet_link" link2="caster_front_right_link" reason="Never"/>
+        <disable_collisions link1="cabinet_link" link2="wheel_back_link" reason="Never"/>
+        <disable_collisions link1="cabinet_link" link2="wheel_front_left_link" reason="Never"/>
+        <disable_collisions link1="cabinet_link" link2="wheel_front_right_link" reason="Never"/>
+        <disable_collisions link1="cabinet_link" link2="${prefix_value}base_link_inertia" reason="Adjacent"/>
+        <disable_collisions link1="cabinet_link" link2="${prefix_value}shoulder_link" reason="Never"/>
+        <disable_collisions link1="lidar_1_link" link2="lidar_2_link" reason="Adjacent"/>
+        <disable_collisions link1="lidar_1_link" link2="caster_back_link" reason="Never"/>
+        <disable_collisions link1="lidar_1_link" link2="caster_front_left_link" reason="Never"/>
+        <disable_collisions link1="lidar_1_link" link2="caster_front_right_link" reason="Never"/>
+        <disable_collisions link1="lidar_1_link" link2="wheel_back_link" reason="Never"/>
+        <disable_collisions link1="lidar_1_link" link2="wheel_front_left_link" reason="Never"/>
+        <disable_collisions link1="lidar_1_link" link2="wheel_front_right_link" reason="Never"/>
+        <disable_collisions link1="lidar_1_link" link2="${prefix_value}base_link_inertia" reason="Never"/>
+        <disable_collisions link1="lidar_1_link" link2="${prefix_value}shoulder_link" reason="Never"/>
+        <disable_collisions link1="lidar_2_link" link2="caster_back_link" reason="Never"/>
+        <disable_collisions link1="lidar_2_link" link2="caster_front_left_link" reason="Never"/>
+        <disable_collisions link1="lidar_2_link" link2="caster_front_right_link" reason="Never"/>
+        <disable_collisions link1="lidar_2_link" link2="wheel_back_link" reason="Never"/>
+        <disable_collisions link1="lidar_2_link" link2="wheel_front_left_link" reason="Never"/>
+        <disable_collisions link1="lidar_2_link" link2="wheel_front_right_link" reason="Never"/>
+        <disable_collisions link1="lidar_2_link" link2="${prefix_value}base_link_inertia" reason="Never"/>
+        <disable_collisions link1="lidar_2_link" link2="${prefix_value}shoulder_link" reason="Never"/>
+        <disable_collisions link1="lidar_2_link" link2="${prefix_value}upper_arm_link" reason="Never"/>
+        <disable_collisions link1="caster_back_link" link2="caster_front_left_link" reason="Never"/>
+        <disable_collisions link1="caster_back_link" link2="caster_front_right_link" reason="Never"/>
+        <disable_collisions link1="caster_back_link" link2="wheel_back_link" reason="Adjacent"/>
+        <disable_collisions link1="caster_back_link" link2="wheel_front_left_link" reason="Never"/>
+        <disable_collisions link1="caster_back_link" link2="wheel_front_right_link" reason="Never"/>
+        <disable_collisions link1="caster_back_link" link2="${prefix_value}base_link_inertia" reason="Never"/>
+        <disable_collisions link1="caster_back_link" link2="${prefix_value}shoulder_link" reason="Never"/>
+        <disable_collisions link1="caster_back_link" link2="${prefix_value}upper_arm_link" reason="Never"/>
+        <disable_collisions link1="caster_front_left_link" link2="caster_front_right_link" reason="Never"/>
+        <disable_collisions link1="caster_front_left_link" link2="wheel_back_link" reason="Never"/>
+        <disable_collisions link1="caster_front_left_link" link2="wheel_front_left_link" reason="Adjacent"/>
+        <disable_collisions link1="caster_front_left_link" link2="wheel_front_right_link" reason="Never"/>
+        <disable_collisions link1="caster_front_left_link" link2="${prefix_value}base_link_inertia" reason="Never"/>
+        <disable_collisions link1="caster_front_left_link" link2="${prefix_value}shoulder_link" reason="Never"/>
+        <disable_collisions link1="caster_front_right_link" link2="wheel_back_link" reason="Never"/>
+        <disable_collisions link1="caster_front_right_link" link2="wheel_front_left_link" reason="Never"/>
+        <disable_collisions link1="caster_front_right_link" link2="wheel_front_right_link" reason="Adjacent"/>
+        <disable_collisions link1="caster_front_right_link" link2="${prefix_value}base_link_inertia" reason="Never"/>
+        <disable_collisions link1="caster_front_right_link" link2="${prefix_value}shoulder_link" reason="Never"/>
+        <disable_collisions link1="wheel_back_link" link2="wheel_front_left_link" reason="Never"/>
+        <disable_collisions link1="wheel_back_link" link2="wheel_front_right_link" reason="Never"/>
+        <disable_collisions link1="wheel_back_link" link2="${prefix_value}base_link_inertia" reason="Never"/>
+        <disable_collisions link1="wheel_back_link" link2="${prefix_value}shoulder_link" reason="Never"/>
+        <disable_collisions link1="wheel_back_link" link2="${prefix_value}upper_arm_link" reason="Never"/>
+        <disable_collisions link1="wheel_front_left_link" link2="wheel_front_right_link" reason="Never"/>
+        <disable_collisions link1="wheel_front_left_link" link2="${prefix_value}base_link_inertia" reason="Never"/>
+        <disable_collisions link1="wheel_front_left_link" link2="${prefix_value}shoulder_link" reason="Never"/>
+        <disable_collisions link1="wheel_front_left_link" link2="${prefix_value}upper_arm_link" reason="Never"/>
+        <disable_collisions link1="wheel_front_right_link" link2="${prefix_value}base_link_inertia" reason="Never"/>
+        <disable_collisions link1="wheel_front_right_link" link2="${prefix_value}shoulder_link" reason="Never"/>
+        <disable_collisions link1="wheel_front_right_link" link2="${prefix_value}upper_arm_link" reason="Never"/>
+        <disable_collisions link1="${prefix_value}base_link_inertia" link2="${prefix_value}shoulder_link" reason="Adjacent"/>
+        <disable_collisions link1="${prefix_value}base_link_inertia" link2="${prefix_value}upper_arm_link" reason="Never"/>
+        <disable_collisions link1="${prefix_value}base_link_inertia" link2="${prefix_value}wrist_1_link" reason="Never"/>
+        <disable_collisions link1="${prefix_value}forearm_link" link2="${prefix_value}upper_arm_link" reason="Adjacent"/>
+        <disable_collisions link1="${prefix_value}forearm_link" link2="${prefix_value}wrist_1_link" reason="Adjacent"/>
+        <disable_collisions link1="${prefix_value}shoulder_link" link2="${prefix_value}upper_arm_link" reason="Adjacent"/>
+        <disable_collisions link1="${prefix_value}shoulder_link" link2="${prefix_value}wrist_1_link" reason="Never"/>
+        <disable_collisions link1="${prefix_value}shoulder_link" link2="${prefix_value}wrist_2_link" reason="Never"/>
+        <disable_collisions link1="${prefix_value}wrist_1_link" link2="${prefix_value}wrist_2_link" reason="Adjacent"/>
+        <disable_collisions link1="${prefix_value}wrist_1_link" link2="${prefix_value}wrist_3_link" reason="Never"/>
+        <disable_collisions link1="${prefix_value}wrist_2_link" link2="${prefix_value}wrist_3_link" reason="Adjacent"/>
+        <disable_collisions link1="${prefix_value}tool0" link2="${prefix_value}wrist_1_link" reason="Never" />
+        <disable_collisions link1="${prefix_value}tool0" link2="${prefix_value}wrist_2_link" reason="Never" />
+        <disable_collisions link1="${prefix_value}tool0" link2="${prefix_value}wrist_3_link" reason="Adjacent" />
+    </xacro:if>
 </robot>
