Commit message: adding linear axis

File: neo_rox_moveit2/srdf/rox.srdf.xacro (robot description, xacro)
@@ -42,4 +42,16 @@
     <joint name="${prefix_value}wrist_3_joint" value="4.75" />
   </group_state>
+  <group name="linear_axis">
+      <link name="linear_axis_slide_link"/>
+      <joint name="linear_axis_slide_joint"/>
+      <chain base_link="base_link" tip_link="linear_axis"/>
+  </group>
+  <!--GROUP STATES: Purpose: Define a named state for a particular group, in terms of joint values. This is useful to define states like 'folded arms'-->
+  <group_state name="top" group="linear_axis">
+      <joint name="linear_axis_slide_joint" value="0.68"/>
+  </group_state>
+  <group_state name="down" group="linear_axis">
+      <joint name="linear_axis_slide_joint" value="0.1"/>
+  </group_state>
   <!--DISABLE COLLISIONS: By default it is assumed that any link of the robot could potentially come into collision with any other link in the robot. This tag disables collision checking between a specified pair of links. -->
   <!-- Common collisions for all rox drives-->
@@ -47,4 +59,6 @@
   <disable_collisions link1="base_footprint" link2="lidar_1_link" reason="Adjacent"/>
   <disable_collisions link1="base_footprint" link2="lidar_2_link" reason="Adjacent"/>
+  <disable_collisions link1="base_footprint" link2="linear_axis" reason="Never"/>
+  <disable_collisions link1="base_footprint" link2="linear_axis_slide_link" reason="Adjacent"/>
   <disable_collisions link1="base_footprint" link2="${prefix_value}base_link_inertia" reason="Never"/>
   <disable_collisions link1="base_footprint" link2="${prefix_value}shoulder_link" reason="Never"/>
@@ -74,4 +88,12 @@
   <disable_collisions link1="${prefix_value}tool0" link2="${prefix_value}wrist_2_link" reason="Never" />
   <disable_collisions link1="${prefix_value}tool0" link2="${prefix_value}wrist_3_link" reason="Adjacent" />
+  <disable_collisions link1="${prefix_value}base_link_inertia" link2="linear_axis_link" reason="Never"/>
+  <disable_collisions link1="${prefix_value}shoulder_link" link2="linear_axis_link" reason="Never"/>
+  <disable_collisions link1="${prefix_value}upper_arm_link" link2="linear_axis_link" reason="Never"/>
+  <disable_collisions link1="${prefix_value}forearm_link" link2="linear_axis_link" reason="Never"/>
+  <disable_collisions link1="${prefix_value}wrist_1_link" link2="linear_axis_link" reason="Never"/>
+  <disable_collisions link1="${prefix_value}wrist_2_link" link2="linear_axis_link" reason="Never"/>
+  <disable_collisions link1="${prefix_value}wrist_3_link" link2="linear_axis_link" reason="Never"/>
+  <disable_collisions link1="${prefix_value}tool0" link2="linear_axis_link" reason="Never"/>
   <xacro:if value="${rox_typ == 'argo' or rox_typ == 'argo-trio'}">
     <xacro:include filename="$(find neo_rox_moveit2)/srdf/rox_argo.srdf.xacro" />

File: neo_rox_moveit2/srdf/rox_argo.srdf.xacro (robot description, xacro)
@@ -43,4 +43,12 @@
     <disable_collisions link1="wheel_front_right_link" link2="${prefix_value}shoulder_link" reason="Never"/>
     <disable_collisions link1="wheel_front_right_link" link2="${prefix_value}upper_arm_link" reason="Never"/>
+    <disable_collisions link1="base_footprint" link2="linear_axis_link" reason="Never"/>
+    <disable_collisions link1="cabinet_link" link2="linear_axis_link" reason="Never"/>
+    <disable_collisions link1="lidar_1_link" link2="linear_axis_link" reason="Never"/>
+    <disable_collisions link1="lidar_2_link" link2="linear_axis_link" reason="Never"/>
+    <disable_collisions link1="caster_front_left_link" link2="linear_axis_link" reason="Never"/>
+    <disable_collisions link1="caster_front_right_link" link2="linear_axis_link" reason="Never"/>
+    <disable_collisions link1="wheel_front_left_link" link2="linear_axis_link" reason="Never"/>
+    <disable_collisions link1="wheel_front_right_link" link2="linear_axis_link" reason="Never"/>
     <xacro:if value="${rox_typ == 'argo'}">
       <disable_collisions link1="base_footprint" link2="caster_back_left_link" reason="Adjacent"/>
@@ -94,4 +102,16 @@
       <disable_collisions link1="wheel_back_right_link" link2="${prefix_value}shoulder_link" reason="Never"/>
       <disable_collisions link1="wheel_back_right_link" link2="${prefix_value}upper_arm_link" reason="Never"/>
+      <disable_collisions link1="base_footprint" link2="linear_axis_link" reason="Never"/>
+      <disable_collisions link1="cabinet_link" link2="linear_axis_link" reason="Never"/>
+      <disable_collisions link1="lidar_1_link" link2="linear_axis_link" reason="Never"/>
+      <disable_collisions link1="lidar_2_link" link2="linear_axis_link" reason="Never"/>
+      <disable_collisions link1="caster_front_left_link" link2="linear_axis_link" reason="Never"/>
+      <disable_collisions link1="caster_front_right_link" link2="linear_axis_link" reason="Never"/>
+      <disable_collisions link1="wheel_front_left_link" link2="linear_axis_link" reason="Never"/>
+      <disable_collisions link1="wheel_front_right_link" link2="linear_axis_link" reason="Never"/>
+      <disable_collisions link1="caster_back_left_link" link2="linear_axis_link" reason="Never"/>
+      <disable_collisions link1="caster_back_right_link" link2="linear_axis_link" reason="Never"/>
+      <disable_collisions link1="wheel_back_left_link" link2="linear_axis_link" reason="Never"/>
+      <disable_collisions link1="wheel_back_right_link" link2="linear_axis_link" reason="Never"/>
     </xacro:if>
     <xacro:if value="${rox_typ == 'argo-trio'}">

Commit message: updates for the linear axis

File: neo_rox_moveit2/srdf/rox.srdf.xacro (robot description, xacro)
@@ -26,24 +26,16 @@
   </group>
   <!--GROUP STATES: Purpose: Define a named state for a particular group, in terms of joint values. This is useful to define states like 'folded arms'-->
-  <group_state name="up" group="ur_manipulator">
-    <joint name="${prefix_value}elbow_joint" value="0" />
-    <joint name="${prefix_value}shoulder_lift_joint" value="-1.5707" />
-    <joint name="${prefix_value}shoulder_pan_joint" value="0" />
-    <joint name="${prefix_value}wrist_1_joint" value="-1.5707" />
-    <joint name="${prefix_value}wrist_2_joint" value="0" />
-    <joint name="${prefix_value}wrist_3_joint" value="0" />
-  </group_state>
-  <group_state name="test_configuration" group="ur_manipulator">
-    <joint name="${prefix_value}elbow_joint" value="1.83" />
-    <joint name="${prefix_value}shoulder_lift_joint" value="-2.66" />
-    <joint name="${prefix_value}shoulder_pan_joint" value="3.14" />
-    <joint name="${prefix_value}wrist_1_joint" value="-1.45" />
-    <joint name="${prefix_value}wrist_2_joint" value="3.22" />
-    <joint name="${prefix_value}wrist_3_joint" value="4.75" />
+  <group_state name="home" group="ur_manipulator">
+    <joint name="${prefix_value}elbow_joint" value="0.112" />
+    <joint name="${prefix_value}shoulder_lift_joint" value="-2.775" />
+    <joint name="${prefix_value}shoulder_pan_joint" value="3.622" />
+    <joint name="${prefix_value}wrist_1_joint" value="-3.020" />
+    <joint name="${prefix_value}wrist_2_joint" value="0.065" />
+    <joint name="${prefix_value}wrist_3_joint" value="0.203" />
   </group_state>
   <group name="linear_axis">
       <link name="linear_axis_slide_link"/>
       <joint name="linear_axis_slide_joint"/>
-      <chain base_link="base_link" tip_link="linear_axis"/>
+      <chain base_link="base_link" tip_link="linear_axis_slide_link"/>
   </group>
   <!--GROUP STATES: Purpose: Define a named state for a particular group, in terms of joint values. This is useful to define states like 'folded arms'-->
@@ -71,4 +63,5 @@
   <disable_collisions link1="cabinet_link" link2="lidar_1_link" reason="Adjacent"/>
   <disable_collisions link1="cabinet_link" link2="lidar_2_link" reason="Adjacent"/>
+  <disable_collisions link1="cabinet_link" link2="linear_axis_fixed_link" reason="Adjacent"/>
   <disable_collisions link1="cabinet_link" link2="${prefix_value}base_link_inertia" reason="Adjacent"/>
   <disable_collisions link1="cabinet_link" link2="${prefix_value}shoulder_link" reason="Never"/>
@@ -88,12 +81,5 @@
   <disable_collisions link1="${prefix_value}tool0" link2="${prefix_value}wrist_2_link" reason="Never" />
   <disable_collisions link1="${prefix_value}tool0" link2="${prefix_value}wrist_3_link" reason="Adjacent" />
-  <disable_collisions link1="${prefix_value}base_link_inertia" link2="linear_axis_link" reason="Never"/>
-  <disable_collisions link1="${prefix_value}shoulder_link" link2="linear_axis_link" reason="Never"/>
-  <disable_collisions link1="${prefix_value}upper_arm_link" link2="linear_axis_link" reason="Never"/>
-  <disable_collisions link1="${prefix_value}forearm_link" link2="linear_axis_link" reason="Never"/>
-  <disable_collisions link1="${prefix_value}wrist_1_link" link2="linear_axis_link" reason="Never"/>
-  <disable_collisions link1="${prefix_value}wrist_2_link" link2="linear_axis_link" reason="Never"/>
-  <disable_collisions link1="${prefix_value}wrist_3_link" link2="linear_axis_link" reason="Never"/>
-  <disable_collisions link1="${prefix_value}tool0" link2="linear_axis_link" reason="Never"/>
+  <disable_collisions link1="${prefix_value}base_link_inertia" link2="linear_axis_slide_link" reason="Never"/>
   <xacro:if value="${rox_typ == 'argo' or rox_typ == 'argo-trio'}">
     <xacro:include filename="$(find neo_rox_moveit2)/srdf/rox_argo.srdf.xacro" />

File: neo_rox_moveit2/srdf/rox_argo.srdf.xacro (robot description, xacro)
@@ -43,12 +43,5 @@
     <disable_collisions link1="wheel_front_right_link" link2="${prefix_value}shoulder_link" reason="Never"/>
     <disable_collisions link1="wheel_front_right_link" link2="${prefix_value}upper_arm_link" reason="Never"/>
-    <disable_collisions link1="base_footprint" link2="linear_axis_link" reason="Never"/>
-    <disable_collisions link1="cabinet_link" link2="linear_axis_link" reason="Never"/>
-    <disable_collisions link1="lidar_1_link" link2="linear_axis_link" reason="Never"/>
-    <disable_collisions link1="lidar_2_link" link2="linear_axis_link" reason="Never"/>
-    <disable_collisions link1="caster_front_left_link" link2="linear_axis_link" reason="Never"/>
-    <disable_collisions link1="caster_front_right_link" link2="linear_axis_link" reason="Never"/>
-    <disable_collisions link1="wheel_front_left_link" link2="linear_axis_link" reason="Never"/>
-    <disable_collisions link1="wheel_front_right_link" link2="linear_axis_link" reason="Never"/>
+    <disable_collisions link1="linear_axis_fixed_link" link2="linear_axis_slide_link" reason="Never"/>
     <xacro:if value="${rox_typ == 'argo'}">
       <disable_collisions link1="base_footprint" link2="caster_back_left_link" reason="Adjacent"/>
@@ -102,16 +95,4 @@
       <disable_collisions link1="wheel_back_right_link" link2="${prefix_value}shoulder_link" reason="Never"/>
       <disable_collisions link1="wheel_back_right_link" link2="${prefix_value}upper_arm_link" reason="Never"/>
-      <disable_collisions link1="base_footprint" link2="linear_axis_link" reason="Never"/>
-      <disable_collisions link1="cabinet_link" link2="linear_axis_link" reason="Never"/>
-      <disable_collisions link1="lidar_1_link" link2="linear_axis_link" reason="Never"/>
-      <disable_collisions link1="lidar_2_link" link2="linear_axis_link" reason="Never"/>
-      <disable_collisions link1="caster_front_left_link" link2="linear_axis_link" reason="Never"/>
-      <disable_collisions link1="caster_front_right_link" link2="linear_axis_link" reason="Never"/>
-      <disable_collisions link1="wheel_front_left_link" link2="linear_axis_link" reason="Never"/>
-      <disable_collisions link1="wheel_front_right_link" link2="linear_axis_link" reason="Never"/>
-      <disable_collisions link1="caster_back_left_link" link2="linear_axis_link" reason="Never"/>
-      <disable_collisions link1="caster_back_right_link" link2="linear_axis_link" reason="Never"/>
-      <disable_collisions link1="wheel_back_left_link" link2="linear_axis_link" reason="Never"/>
-      <disable_collisions link1="wheel_back_right_link" link2="linear_axis_link" reason="Never"/>
     </xacro:if>
     <xacro:if value="${rox_typ == 'argo-trio'}">
